Commit message: P1: geometria del robot en una sola fuente de verdad (YAML + xacro)
Las dimensiones fisicas estaban duplicadas e independientes entre el URDF y
kinematic_guardian, ya desincronizadas (largo del flipper: 0.265 en el guardian
vs 0.26 en el URDF). Actualizar las medidas reales exigia tocar ~15 valores en
dos formatos distintos.

Ahora config/geometria_robot.yaml es la unica fuente:
  - urdf/ugv.urdf.xacro la lee con xacro.load_yaml y reemplaza los 4 bloques de
    flipper copiados por una macro instanciada 4 veces. Los launch procesan el
    xacro en caliente, asi que el modelo no puede quedar desfasado.
  - kinematic_guardian recibe distancia_motor_x/z, largo_flipper y
    radio_rueda_flipper por declare_parameter. El algoritmo geometrico
    (interseccion de segmentos + distancia punto-segmento) queda intacto.
  - track_odometry_node y el driver toman radio_oruga/ancho_orugas del mismo
    archivo (antes duplicados entre ambos).

El umbral de proximidad del guardian pasa de la constante 0.0324 a
(2*radio_rueda_flipper)^2, que da el mismo 0.0324 pero derivado: es la suma de
radios de las dos capsulas, y ya no puede desincronizarse del URDF.
Unificado el largo del flipper en 0.26 (el guardian queda 5 mm menos
conservador que antes, ahora coincidiendo con la geometria real dibujada).

scripts/generar_urdf.sh regenera el .urdf plano para Foxglove y herramientas
que no procesan xacro. Verificado: el URDF generado es geometricamente identico
al anterior (solo cambia la precision de pi/2) y el TF resultante coincide.

Ademas, dos arreglos que venian pegados:
  - base_link ya no lleva <inertial> (su masa pasa a chassis_inertial_link, hijo
    fijo): elimina el warning de kdl_parser en cada arranque de
    robot_state_publisher. NO se uso el truco del dummy_link como raiz porque
    dejaria base_link con dos padres (dummy_link y el odom->base_link del EKF),
    invalidando el arbol TF.
  - setup.py registraba gui_a_vcan y dummy_rl_controller, dos modulos que no
    existen, y no registraba gui_a_comandos ni can_monitor, que si existen y son
    invocados por can_view.launch.py y can_studio.launch.py: esos dos launch
    estaban rotos.

Co-Authored-By: Claude Opus 5 <noreply@anthropic.com>

File: src/ugv_bridge/urdf/ugv.urdf (robot description, URDF)
Before this commit: robot ugv_MARV, 6 links, 5 joints
Links:
- added link chassis_inertial_link, mass 20.0
- link base_link: mass 20.0 -> None; geometry collision box size=0.6 0.36 0.2; visual mesh filename=package://ugv_bridge/meshes/chassis.dae scale=1 1 1
Joints:
- added joint chassis_inertial_joint: type fixed, parent base_link, child chassis_inertial_link, origin xyz=0 0 0 rpy=0 0 0
- joint flipper_rl: origin xyz=-0.23 0.195 -0.03 rpy=0 0 3.14159 -> xyz=-0.23 0.195 -0.03 rpy=0 0 3.141592653589793
- joint flipper_rr: origin xyz=-0.23 -0.195 -0.03 rpy=0 0 3.14159 -> xyz=-0.23 -0.195 -0.03 rpy=0 0 3.141592653589793
